File: MacropadRP2040.kicad_pcb (KiCad board)
At the start: 2 copper layers, 95 x 45 mm, 27 parts, among them Q1 AO3400A, SW1 SW_Push, SW2 SW_Push, SW3 SW_Push, SW4 RotaryEncoder_Switch_MP, SW5 SW_Push, SW6 SW_Push, SW7 SW_Push, U1 RP2040-ZERO

Commit message: PCB todo
Parts:
- D10, D7, D8, D9, Q1, R3, R4: moved to F.Cu
- SW4: value RotaryEncoder_Switch_MP -> SW_Push
- SW7: value SW_Push -> RotaryEncoder_Switch_MP
- moved Q1 27.2 mm to (51.0, 8.44)
- moved R3 27.2 mm to (51.0, 12.4)
- moved R4 27.2 mm to (51.0, 4.19)
- moved R2 8.57 mm to (59.8, 21.5), turned to 90 degrees
- moved SW7 7.00 mm to (71.2, 23.8)
- moved R1 1.17 mm to (67.0, 21.4), turned to 90 degrees
- moved D9 0.55 mm to (-10.2, 9.50), turned to -90 degrees
- moved D6 0.50 mm to (28.5, 20.5)
- turned D7 to -90 degrees
Connections:
- D1 pad 1: colunm1 -> row1
- D2 pad 1: colunm1 -> row1
- D3 pad 1: colunm1 -> row1
- D4 pad 1: colunm1 -> row2
- D5 pad 1: colunm1 -> row2
- D6 pad 1: colunm1 -> row2
- SW1 pad 2: colunm1 -> column1
- SW2 pad 2: colunm1 -> column2
- SW3 pad 2: colunm1 -> column3
- SW4 pad 1: (no net) -> Net-(D4-A)
- SW4 pad 2: (no net) -> column1
- SW5 pad 1: Net-(D4-A) -> Net-(D5-A)
- SW5 pad 2: colunm1 -> column2
- SW6 pad 1: Net-(D5-A) -> Net-(D6-A)
- SW6 pad 2: colunm1 -> column3
- SW7 pad A: (no net) -> clk_enc
- SW7 pad B: (no net) -> dt_enc
- SW7 pad C: (no net) -> GND
- SW7 pad MP: (no net) -> GND
- SW7 pad S1: (no net) -> sw_enc
- SW7 pad S2: (no net) -> GND
- U1 pad 1: colunm1 -> row1
- U1 pad 2: colunm1 -> row2
- U1 pad 21: unconnected-(U1-3V3-Pad21) -> +3V3
- U1 pad 3: colunm1 -> column1
- U1 pad 4: colunm1 -> column2
- U1 pad 5: colunm1 -> column3
Routing:
- net row2: track 0.00 -> 246.0 mm
- net column1: track 0.00 -> 169.2 mm
- net +5V: track 19.9 -> 182.6 mm, vias 0 -> 1
- net column2: track 0.00 -> 111.2 mm
- net column3: track 0.00 -> 89.9 mm
- net GND: track 53.6 -> 137.8 mm
- net row1: track 0.00 -> 81.1 mm, vias 0 -> 2
- net Net-(D8-DOUT): track 0.00 -> 69.9 mm
- net Net-(D10-DIN): track 0.00 -> 57.3 mm
- net Net-(D7-DOUT): track 0.00 -> 56.3 mm
- net colunm1: track 40.0 -> 0.00 mm
- net Net-(D7-DIN): track 3.69 -> 33.6 mm
- net +3V3: track 11.6 -> 30.4 mm, vias 0 -> 1
- net dt_enc: track 15.3 -> 24.5 mm
- net led_rgb: track 19.5 -> 24.0 mm, vias 0 -> 1
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
Commit message: zones added
Signed-off-by: BrendonBernardino <brendonrsb@hotmail.com>
Parts:
- moved D10 20.0 mm to (47.6, 42.8)
- moved R1 19.2 mm to (81.1, 34.4)
- moved SW4 19.2 mm to (14.1, 32.0)
- moved SW5 19.2 mm to (33.1, 32.0)
- moved SW6 19.2 mm to (52.2, 32.0)
- moved C1 19.2 mm to (65.7, 10.5)
- moved C2 19.2 mm to (65.7, 8.48)
- moved C3 19.2 mm to (65.7, 6.48)
- moved C4 19.2 mm to (65.7, 4.45)
- moved D1 19.2 mm to (4.58, 14.7)
- moved D2 19.2 mm to (23.6, 15.0)
- moved D3 19.2 mm to (42.6, 15.0)
- moved D4 19.2 mm to (4.58, 33.5)
- moved D7 19.2 mm to (89.8, 22.5)
- moved D9 19.2 mm to (3.88, 22.5)
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Routing:
- net row1: track 81.1 -> 284.1 mm
- net +5V: track 182.6 -> 263.4 mm
- net GND: track 137.8 -> 147.6 mm, vias 0 -> 2
- net column1: track 169.2 -> 177.4 mm
- net Net-(D7-DOUT): track 56.3 -> 64.2 mm
- net row2: track 246.0 -> 251.2 mm
- net column2: track 111.2 -> 114.0 mm
- net column3: track 89.9 -> 92.6 mm
- net Net-(D10-DIN): track 57.3 -> 58.6 mm
- net +3V3: track 30.4 -> 31.2 mm
- net Net-(D7-DIN): track 33.6 -> 32.8 mm
- net sw_enc: track 10.2 -> 10.8 mm
- net clk_enc: track 28.7 -> 29.4 mm
- net led_rgb: track 24.0 -> 24.7 mm
- added copper zone on B.Cu, net +5V
- added copper zone on F.Cu, net GND
Other:
- board size 95 x 45 mm -> 95 x 48 mm
- board text added: "Po1son.bit"
