File: MacropadRP2040.kicad_pcb (KiCad board)
At the start: 2 copper layers, 95 x 45 mm, 27 parts, among them Q1 AO3400A, SW1 SW_Push, SW2 SW_Push, SW3 SW_Push, SW4 SW_Push, SW5 SW_Push, SW6 SW_Push, SW7 RotaryEncoder_Switch_MP, U1 RP2040-ZERO

Commit message: zones added
Signed-off-by: BrendonBernardino <brendonrsb@hotmail.com>
Parts:
- moved R1 19.2 mm to (81.1, 34.4)
- moved SW4 19.2 mm to (14.1, 32.0)
- moved SW5 19.2 mm to (33.1, 32.0)
- moved SW6 19.2 mm to (52.2, 32.0)
- moved C1 19.2 mm to (65.7, 10.5)
- moved C2 19.2 mm to (65.7, 8.48)
- moved C3 19.2 mm to (65.7, 6.48)
- moved C4 19.2 mm to (65.7, 4.45)
- moved D1 19.2 mm to (4.58, 14.7)
- moved D2 19.2 mm to (23.6, 15.0)
- moved D3 19.2 mm to (42.6, 15.0)
- moved D4 19.2 mm to (4.58, 33.5)
- moved D7 19.2 mm to (89.8, 22.5)
- moved D8 19.2 mm to (47.6, 3.23)
- moved D9 19.2 mm to (3.88, 22.5)
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Routing:
- net row1: track 81.1 -> 277.6 mm
- net +5V: track 182.6 -> 210.7 mm
- net GND: track 137.8 -> 165.6 mm, vias 0 -> 2
- net column1: track 169.2 -> 172.6 mm
- net Net-(D8-DOUT): track 69.9 -> 69.3 mm
- added copper zone on B.Cu, net +5V
- added copper zone on F.Cu, net GND
Other:
- outline, holes or cut-outs redrawn
